File: Projects/Novice/Novice.kicad_sch (KiCad schematic)
At the start: 4 parts

Commit message: 20240212
Parts:
- removed R2: R, Resistor_THT:R_Axial_DIN0207_L6.3mm_D2.5mm_P7.62mm_Horizontal, symbol Device:R
- added SW1: M2011S3A1W03, symbol 001_user_library:M2011S3A1W03
Other:
- note added: "proba szoveg"
Changed lines of the file:
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@@
     (stroke (width 0) (type default))
+  )
+  (text "proba szoveg" (at 152.335 98.0162 0)
+    (effects (font (size 1.27 1.27) (color 0 132 132 1)) (justify left bottom))
   )
   (symbol (lib_id "Device:LED") (at 154 90 90) (unit 1)
@@
         (path "/ee0b424c-6d87-43cd-b5c8-52715f1d7ee4"
           (reference "BT1") (unit 1)
-        )
-      )
-    )
-  )
-  (symbol (lib_id "Device:R") (at 165.0816 82.5667 0) (mirror y) (unit 1)
-    (in_bom yes) (on_board yes) (dnp no)
-    (property "Reference" "R2" (at 163.1716 81.2967 0)
-      (effects (font (size 1.27 1.27)) (justify left))
-    )
-    (property "Value" "R" (at 163.1716 83.8367 0)
-      (effects (font (size 1.27 1.27)) (justify left))
-    )
-    (property "Footprint" "Resistor_THT:R_Axial_DIN0207_L6.3mm_D2.5mm_P7.62mm_Horizontal" (at 166.8596 82.5667 90)
-      (effects (font (size 1.27 1.27)) hide)
-    )
-    (property "Datasheet" "~" (at 165.0816 82.5667 0)
-      (effects (font (size 1.27 1.27)) hide)
-    )
-    (pin "2")
-    (pin "1")
-    (instances
-      (project "Novice"
-        (path "/ee0b424c-6d87-43cd-b5c8-52715f1d7ee4"
-          (reference "R2") (unit 1)
         )
       )
@@
         )
       )
+    )
+  )
+  (symbol (lib_id "001_user_library:M2011S3A1W03") (at 109.22 88.9 0) (unit 1)
+    (in_bom yes) (on_board yes) (dnp no) (fields_autoplaced)
+    (property "Reference" "SW1" (at 109.22 81.28 0)
+      (effects (font (size 1.27 1.27)))
+    )
+    (property "Value" "M2011S3A1W03" (at 109.22 83.82 0)
+      (effects (font (size 1.27 1.27)))
+    )
+    (property "Footprint" "" (at 109.22 88.9 0)
+      (effects (font (size 1.27 1.27)) hide)
+    )
+    (property "Datasheet" "" (at 109.22 88.9 0)
+      (effects (font (size 1.27 1.27)) hide)
+    )
+    (pin "2")
+    (pin "3")
+    (instances
+      (project "Novice"
+        (path "/ee0b424c-6d87-43cd-b5c8-52715f1d7ee4"
+          (reference "SW1") (unit 1)
+        )
+      )

Commit message: 20240214
Parts:
- removed SW1: M2011S3A1W03, symbol 001_user_library:M2011S3A1W03
- added K1, K2: M2011S3A1W03, helyi_sajat:kapcsolo, symbol user-novice:M2011S3A1W03
Connections:
- net VCC: now also K1.3 (B); no longer BT1.1 (+)
- new net: BT1.1 (+), K1.2 (A)
Other:
- moved on the sheet: BT1, R1
