File: Projects/Sidetone/Sidetone-javitott.kicad_pcb (KiCad board)
At the start: 2 copper layers, 109.1 x 105 mm, 54 parts, among them Q1 2N3904, Q2 2N3904, Q3 2N3904, SW1 morse key, SW2 On/off, U1 4N35, U2 LM324, U3 LM386

Commit message: 20240302
Connections:
- 4-8ohm1 pad 2: GNDD -> Net-(D3-K)
- C1 pad 1: Net-(U2A--) -> Net-(D3-K)
- C1 pad 2: GNDD -> Net-(D3-K)
- C11 pad 2: GNDD -> Net-(D3-K)
- C2 pad 1: Net-(Q2-B) -> Net-(D3-K)
- C2 pad 2: GNDD -> Net-(D3-K)
- C5 pad 2: GNDD -> Net-(D3-K)
- C6 pad 1: Net-(Q1-C) -> Net-(D3-K)
- C7 pad 2: GNDD -> Net-(D3-K)
- C8 pad 2: Net-(C8-Pad2) -> Net-(D3-K)
- C9 pad 2: GNDD -> Net-(D3-K)
- D3 pad 2: GNDD -> Net-(D3-K)
- GND1 pad 1: GNDD -> Net-(D3-K)
- Q1 pad 2: Net-(Q1-B) -> Net-(D3-K)
- Q1 pad 3: Net-(Q1-C) -> Net-(D3-K)
- Q2 pad 2: Net-(Q2-B) -> Net-(D3-K)
- Q3 pad 2: Net-(Q3-B) -> Net-(D3-K)
- Q3 pad 3: Net-(Q3-C) -> Net-(D3-K)
- R10 pad 1: Net-(Q1-B) -> Net-(D3-K)
- R11 pad 2: Net-(Q1-C) -> Net-(D3-K)
- R12 pad 2: GNDD -> Net-(D3-K)
- R13 pad 2: Net-(Q3-C) -> Net-(D3-K)
- R15 pad 1: Net-(R15-Pad1) -> Net-(D3-K)
- R15 pad 2: Net-(Q3-B) -> Net-(D3-K)
- R17 pad 1: Net-(Q3-C) -> Net-(D3-K)
- R17 pad 2: Net-(R15-Pad1) -> Net-(D3-K)
- R18 pad 2: GNDD -> Net-(D3-K)
- R19 pad 1: Net-(Q1-C) -> Net-(D3-K)
- R2 pad 2: Net-(U2A--) -> Net-(D3-K)
- R22 pad 1: Net-(R22-Pad1) -> Net-(D3-K)
- R23 pad 2: GNDD -> Net-(D3-K)
- R3 pad 1: Net-(U2A--) -> Net-(D3-K)
- R3 pad 2: GNDD -> Net-(D3-K)
- R4 pad 2: Net-(Q2-B) -> Net-(D3-K)
- R5 pad 1: Net-(Q2-B) -> Net-(D3-K)
- R5 pad 2: GNDD -> Net-(D3-K)
- R8 pad 1: Net-(R15-Pad1) -> Net-(D3-K)
- R8 pad 2: Net-(Q1-B) -> Net-(D3-K)
- RV1 pad 1: Net-(C8-Pad2) -> Net-(D3-K)
- RV1 pad 2: Net-(R22-Pad1) -> Net-(D3-K)
- RV1 pad 3: GNDD -> Net-(D3-K)
- SW1 pad 2: GNDD -> Net-(D3-K)
- SW2 pad 2: VCC -> Net-(D3-K)
- U2 pad 11: GNDD -> Net-(D3-K)
- U2 pad 12: Net-(U2A--) -> Net-(D3-K)
- U2 pad 2: Net-(U2A--) -> Net-(D3-K)
- U2 pad 5: Net-(Q3-C) -> Net-(D3-K)
- U2 pad 6: Net-(Q1-C) -> Net-(D3-K)
- U3 pad 2: GNDD -> Net-(D3-K)
- U3 pad 4: GNDD -> Net-(D3-K)
- Vcc1 pad : VCC -> Net-(D3-K)
Routing:
- net Net-(D3-K): track 741.9 -> 2024.3 mm, vias 9 -> 28
- net GNDD: track 464.5 -> 0.00 mm, vias 6 -> 0
- net Net-(Q1-C): track 265.7 -> 0.00 mm, vias 2 -> 0
- net Net-(Q3-C): track 210.3 -> 0.00 mm, vias 1 -> 0
- net Net-(R15-Pad1): track 70.9 -> 0.00 mm, vias 2 -> 0
- net Net-(R22-Pad1): track 70.7 -> 0.00 mm, vias 2 -> 0
- net Net-(U2A--): track 70.2 -> 0.00 mm, vias 2 -> 0
- net Net-(Q1-B): track 44.8 -> 0.00 mm, vias 2 -> 0
- net Net-(Q3-B): track 26.8 -> 0.00 mm, vias 2 -> 0
- net VCC: track 25.8 -> 0.00 mm
- net Net-(Q2-B): track 24.7 -> 0.00 mm
- net Net-(C8-Pad2): track 8.08 -> 0.00 mm
